File: GB_MemoryBackup_Subboard_A/GB_MemoryBackup_Subboard_A.kicad_pcb (KiCad board)
At the start: 2 copper layers, 55.5 x 35 mm, 2 parts, among them J2 GB_Cart_Slot-1Row-32Pins, J4 Conn_02x16_Odd_Even

Commit message: Modified: PCB routed.
Parts:
- added G***: LOGO, LogoGraphics:12mm_x_12mm_ShadowSonic, B.Cu at (169.5, 108.0)
- added G***: LOGO, LogoGraphics:12mm_x_12mm_ShadowSonic, F.Cu at (189.9, 106.0)
- renumbered J4 to J1
Routing:
- net /ACLK: track 0.00 -> 19.7 mm
- net /~ARD_T: track 0.00 -> 11.1 mm
- net GND: track 0.00 -> 10.7 mm
- net /AA0: track 0.00 -> 10.7 mm
- net /~ARST: track 0.00 -> 10.5 mm
- net /AA2: track 0.00 -> 10.5 mm
- net /AD6: track 0.00 -> 10.3 mm
- net /AA4: track 0.00 -> 10.3 mm
- net /AD4: track 0.00 -> 10.1 mm
- net /AA6: track 0.00 -> 10.1 mm
- net /AD2: track 0.00 -> 9.93 mm
- net /AA8: track 0.00 -> 9.91 mm
- net /AD0: track 0.00 -> 9.74 mm
- net /AA10: track 0.00 -> 9.71 mm
- net /AA14: track 0.00 -> 9.55 mm
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- added copper zone on B.Cu, net +5V
- added copper zone on F.Cu, net GND
Other:
- board text added: "1"
- board text added: "2"
- board text added: "31"
- board text added: "32"
